File: mb_adv_1.0.kicad_pcb (KiCad board)
At the start: 2 copper layers, 50 x 54 mm, 10 parts, among them M2 MountingHole_2.1mm, SW2 SW_SP3T, U2 gba_link_cable, U3 BOB-12009

Commit message: Organize repo
Other:
- board text added: "Thank you to: cozydelaney Ashton Herron (Starlark) prof.beans Cilerba Bucket Mouse wheat jerm and you!"
- board text removed: "Thank you to: cozydelaney Ashton Herron (Starlark) prof. beans Cilerba Bucket Mouse wheat jerm and you!"
Changed lines of the file:
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@@
-		)
-	)
-	(gr_text "Thank you to:\ncozydelaney\nAshton Herron (Starlark)\nprof. beans\nCilerba\nBucket Mouse\nwheat jerm\nand you!"
-		(at 130 121.5 270)
-		(layer "B.SilkS")
-		(effects
-			(font
-				(size 1 1)
-				(thickness 0.1)
-			)
-			(justify left bottom mirror)
 		)
 	)
@@
 		)
 	)
+	(gr_text "Thank you to:\ncozydelaney\nAshton Herron (Starlark)\nprof.beans\nCilerba\nBucket Mouse\nwheat jerm\nand you!"
+		(at 130 121.5 270)
+		(layer "B.SilkS")
+		(effects
+			(font
+				(size 1 1)
+				(thickness 0.2)
+				(bold yes)
+			)
+			(justify left bottom mirror)
+		)
+	)

Commit message: update README.md, schematic, and pcb
Connections:
- A1 pad 2: PSI -> PSO
- A1 pad 4: PSO -> PSI
Routing:
- net PSI: track 39.0 -> 52.6 mm, vias 1 -> 0
- net PSO: track 36.1 -> 46.1 mm
Changed lines of the file:
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@@
 			(layers "*.Cu" "*.Mask")
 			(remove_unused_layers no)
-			(net "PSI")
+			(net "PSO")
 			(pinfunction "GPIO1_2")
 			(pintype "bidirectional")
@@
 			(layers "*.Cu" "*.Mask")
 			(remove_unused_layers no)
-			(net "PSO")
+			(net "PSI")
 			(pinfunction "GPIO2_4")
 			(pintype "bidirectional")
@@
 	)
 	(segment
-		(start 151 108.412232)
-		(end 147.697768 105.11)
+		(start 148.406767 112.695)
+		(end 131.695 112.695)
 		(width 0.5)
 		(layer "F.Cu")
@@
 	)
 	(segment
-		(start 135.5 99.857637)
-		(end 135.5 99)
+		(start 131.695 112.695)
+		(end 129.15 110.15)
+		(width 0.5)
+		(layer "F.Cu")
+		(net "PSI")
+	)
+	(segment
+		(start 127.312233 110.15)
+		(end 126.575 109.412767)
 		(width 0.5)
 		(layer "F.Cu")
@@
 	)
 	(segment
-		(start 147.697768 105.11)
-		(end 140.752363 105.11)
+		(start 151 108.81)
+		(end 152.212 110.022)
 		(width 0.5)
 		(layer "F.Cu")
@@
 	)
 	(segment
-		(start 140.752363 105.11)
-		(end 135.5 99.857637)
+		(start 127.312233 110.15)
+		(end 129.15 110.15)
 		(width 0.5)
 		(layer "F.Cu")
 		(net "PSI")
 	)
-	(via
-		(at 135.5 99)
-		(size 0.6)
-		(drill 0.3)
-		(layers "F.Cu" "B.Cu")
+	(segment
+		(start 126.575 109.412767)
+		(end 126.575 89.835)
+		(width 0.5)
+		(layer "F.Cu")
 		(net "PSI")
 	)
 	(segment
-		(start 135.5 99)
-		(end 135.5 91.2)
-		(width 0.5)
-		(layer "B.Cu")
+		(start 152.212 110.022)
+		(end 152.212 111.852027)
+		(width 0.5)
+		(layer "F.Cu")
 		(net "PSI")
 	)
 	(segment
-		(start 135.5 91.2)
-		(end 127.8 83.5)
-		(width 0.5)
-		(layer "B.Cu")
+		(start 152.212 111.852027)
+		(end 151.502027 112.562)
+		(width 0.5)
+		(layer "F.Cu")
 		(net "PSI")
 	)
 	(segment
-		(start 141.65 107.65)
-		(end 132.5 98.5)
+		(start 148.539767 112.562)
+		(end 148.406767 112.695)
+		(width 0.5)
+		(layer "F.Cu")
+		(net "PSI")
+	)
+	(segment
+		(start 151.502027 112.562)
+		(end 148.539767 112.562)
+		(width 0.5)
+		(layer "F.Cu")
+		(net "PSI")
+	)
+	(segment
+		(start 126.575 89.835)
+		(end 127.83 88.58)
+		(width 0.5)
+		(layer "F.Cu")
+		(net "PSI")
+	)
+	(segment
+		(start 151 111.35)
+		(end 147.3 107.65)
 		(width 0.5)
 		(layer "F.Cu")
@@
 	)
 	(segment
-		(start 151 111.35)
-		(end 147.3 107.65)
+		(start 147.3 107.65)
+		(end 133.15 107.65)
 		(width 0.5)
 		(layer "F.Cu")
@@
 	)
 	(segment
-		(start 147.3 107.65)
-		(end 141.65 107.65)
+		(start 133.15 107.65)
+		(end 130 104.5)
 		(width 0.5)
 		(layer "F.Cu")
@@
 	)
 	(via
-		(at 132.5 98.5)
+		(at 130 104.5)
 		(size 0.6)
 		(drill 0.3)
@@
 	)
 	(segment
-		(start 132.5 98.5)
-		(end 132.5 93.28)
+		(start 130 104.5)
+		(end 130 85.67)
 		(width 0.5)
 		(layer "B.Cu")
@@
 	)
 	(segment
-		(start 132.5 93.28)
-		(end 127.8 88.58)
-		(width 0.5)
-		(layer "B.Cu")
+		(start 130 85.67)
+		(end 127.83 83.5)
+		(width 0.5)
+		(layer "B.Cu")

Commit message: update pinout
Connections:
- A1 pad 10: unconnected-(A1-GPIO7-Pad10) -> PSO
- A1 pad 2: PSO -> PSI
- A1 pad 22: unconnected-(A1-GPIO17-Pad22) -> OPT_1
- A1 pad 26: OPT_1 -> PSI
- A1 pad 4: PSI -> PSO
- A1 pad 7: unconnected-(A1-GPIO5-Pad7) -> PSD
- A1 pad 9: unconnected-(A1-GPIO6-Pad9) -> PSC
Routing:
- net PSC: track 30.5 -> 52.8 mm
- net OPT_1: track 32.9 -> 41.1 mm
- net PSI: track 52.6 -> 60.0 mm
- net PSD: track 27.4 -> 33.5 mm
- net PSO: track 46.1 -> 43.5 mm
- net GND: track 53.5 -> 52.1 mm
- net LV: track 31.0 -> 29.9 mm, vias 2 -> 1
Changed lines of the file:
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@@
 			(layers "*.Cu" "*.Mask")
 			(remove_unused_layers no)
-			(net "PSO")
+			(net "PSI")
 			(pinfunction "GPIO1_2")
 			(pintype "bidirectional")
@@
 			(layers "*.Cu" "*.Mask")
 			(remove_unused_layers no)
-			(net "PSI")
+			(net "PSO")
 			(pinfunction "GPIO2_4")
 			(pintype "bidirectional")
@@
 			(layers "*.Cu" "*.Mask")
 			(remove_unused_layers no)
-			(net "unconnected-(A1-GPIO5-Pad7)")
+			(net "PSD")
 			(pinfunction "GPIO5_7")
 			(pintype "bidirectional")
@@
 			(layers "*.Cu" "*.Mask")
 			(remove_unused_layers no)
-			(net "unconnected-(A1-GPIO6-Pad9)")
+			(net "PSC")
 			(pinfunction "GPIO6_9")
 			(pintype "bidirectional")
@@
 			(layers "*.Cu" "*.Mask")
 			(remove_unused_layers no)
-			(net "unconnected-(A1-GPIO7-Pad10)")
+			(net "PSO")
 			(pinfunction "GPIO7_10")
 			(pintype "bidirectional")
@@
 			(layers "*.Cu" "*.Mask")
 			(remove_unused_layers no)
-			(net "unconnected-(A1-GPIO17-Pad22)")
+			(net "OPT_1")
 			(pinfunction "GPIO17_22")
 			(pintype "bidirectional")
@@
 			(layers "*.Cu" "*.Mask")
 			(remove_unused_layers no)
-			(net "OPT_1")
+			(net "PSI")
 			(pinfunction "GPIO20_26")
 			(pintype "bidirectional")
@@
 	)
 	(gr_text "Thank you to:\ncozydelaney\nAshton Herron (Starlark)\nprof.beans\nCilerba\nBucket Mouse\nwheat jerm\nand you!"
-		(at 130 121.5 270)
+		(at 130.62 121.59 270)
 		(layer "B.SilkS")
 		(effects
@@
 	)
 	(segment
-		(start 148 89.867409)
-		(end 148 88.46)
-		(width 0.8)
-		(layer "B.Cu")
-		(net "GND")
-	)
-	(segment
 		(start 151 106.27)
 		(end 150.75 106.27)
@@
 	)
 	(segment
+		(start 158.5 82)
+		(end 154 86.5)
+		(width 0.8)
+		(layer "F.Cu")
+		(net "LV")
+	)
+	(segment
+		(start 154 86.5)
+		(end 154 90.085785)
+		(width 0.8)
+		(layer "F.Cu")
+		(net "LV")
+	)
+	(segment
+		(start 154 90.085785)
+		(end 157.457107 93.542893)
+		(width 0.8)
+		(layer "F.Cu")
+		(net "LV")
+	)
+	(segment
+		(start 160.66 82)
+		(end 158.5 82)
+		(width 0.8)
+		(layer "F.Cu")
+		(net "LV")
+	)
+	(segment
 		(start 157.457107 93.542893)
 		(end 157.457108 93.542893)
 		(width 0.8)
 		(layer "F.Cu")
-		(net "LV")
-	)
-	(segment
-		(start 154 90.085785)
-		(end 157.457107 93.542893)
-		(width 0.8)
-		(layer "F.Cu")
-		(net "LV")
-	)
-	(segment
-		(start 154 84.5)
-		(end 154 90.085785)
-		(width 0.8)
-		(layer "F.Cu")
-		(net "LV")
-	)
-	(via
-		(at 154 84.5)
-		(size 0.6)
-		(drill 0.3)
-		(layers "F.Cu" "B.Cu")
 		(net "LV")
 	)
@@
 	)
 	(segment
-		(start 158.16 84.5)
-		(end 160.66 82)
-		(width 0.8)
-		(layer "B.Cu")
-		(net "LV")
-	)
-	(segment
-		(start 154 84.5)
-		(end 158.16 84.5)
-		(width 0.8)
-		(layer "B.Cu")
-		(net "LV")
-	)
-	(segment
 		(start 157.457107 93.542893)
 		(end 157.457107 97.272893)
@@
 	)
 	(segment
+		(start 127.83 80.96)
+		(end 125.5 83.29)
+		(width 0.5)
+		(layer "F.Cu")
+		(net "PSC")
+	)
+	(segment
 		(start 147.26 94.91)
 		(end 141.75 94.91)
@@
 	)
 	(segment
+		(start 125.5 83.29)
+		(end 125.5 98.95)
+		(width 0.5)
+		(layer "F.Cu")
+		(net "PSC")
+	)
+	(segment
 		(start 141.75 94.91)
 		(end 127.8 80.96)
@@
 	)
 	(segment
+		(start 125.5 98.95)
+		(end 127.83 101.28)
+		(width 0.5)
+		(layer "F.Cu")
+		(net "PSC")
+	)
+	(segment
 		(start 151 101.19)
 		(end 147.295 97.485)
@@
 	)
 	(segment
-		(start 148.406767 112.695)
-		(end 131.695 112.695)
+		(start 127.83 96.2)
+		(end 126.58 94.95)
+		(width 0.5)
+		(layer "B.Cu")
+		(net "PSD")
+	)
+	(segment
+		(start 126.58 92.37)
+		(end 127.83 91.12)
+		(width 0.5)
+		(layer "B.Cu")
+		(net "PSD")
+	)
+	(segment
+		(start 126.58 94.95)
+		(end 126.58 92.37)
+		(width 0.5)
+		(layer "B.Cu")
+		(net "PSD")
+	)
+	(segment
+		(start 147.26 105.07)
+		(end 151 108.81)
 		(width 0.5)
 		(layer "F.Cu")
@@
 	)
 	(segment
-		(start 131.695 112.695)
-		(end 129.15 110.15)
-		(width 0.5)
-		(layer "F.Cu")
-		(net "PSI")
-	)
-	(segment
-		(start 127.312233 110.15)
-		(end 126.575 109.412767)
+		(start 126.575 94.172767)
+		(end 127.312233 94.91)
 		(width 0.5)
 		(layer "F.Cu")
@@
 	)
 	(segment
+		(start 128.347767 94.91)
+		(end 138.507767 105.07)
+		(width 0.5)
+		(layer "F.Cu")
+		(net "PSI")
+	)
+	(segment
+		(start 127.312233 94.91)
+		(end 128.347767 94.91)
+		(width 0.5)
+		(layer "F.Cu")
+		(net "PSI")
+	)
+	(segment
+		(start 138.507767 105.07)
+		(end 147.26 105.07)
+		(width 0.5)
+		(layer "F.Cu")
+		(net "PSI")
+	)
+	(segment
+		(start 126.575 84.755)
+		(end 126.575 94.172767)
+		(width 0.5)
+		(layer "F.Cu")
+		(net "PSI")
+	)
+	(segment
+		(start 127.83 83.5)
+		(end 126.575 84.755)
+		(width 0.5)
+		(layer "F.Cu")
+		(net "PSI")
+	)
+	(segment
+		(start 146.86 115.27)
+		(end 146.86 113.462233)
+		(width 0.5)
+		(layer "B.Cu")
+		(net "PSI")
+	)
+	(segment
+		(start 145.092233 107.65)
+		(end 144.355 108.387233)
+		(width 0.5)
+		(layer "B.Cu")
+		(net "PSI")
+	)
+	(segment
+		(start 144.355 108.387233)
+		(end 144.355 112.311312)
+		(width 0.5)
+		(layer "B.Cu")
+		(net "PSI")
+	)
+	(segment
+		(start 144.355 112.311312)
+		(end 144.773688 112.73)
+		(width 0.5)
+		(layer "B.Cu")
+		(net "PSI")
+	)
+	(segment
+		(start 146.127767 112.73)
+		(end 146.698884 113.301116)
+		(width 0.5)
+		(layer "B.Cu")
+		(net "PSI")
+	)
+	(segment
+		(start 145.61 116.52)
+		(end 146.86 115.27)
+		(width 0.5)
+		(layer "B.Cu")
+		(net "PSI")
+	)
+	(segment
+		(start 146.86 113.462233)
+		(end 146.698884 113.301116)
+		(width 0.5)
+		(layer "B.Cu")
+		(net "PSI")
+	)
+	(segment
 		(start 151 108.81)
-		(end 152.212 110.022)
-		(width 0.5)
-		(layer "F.Cu")
+		(end 149.84 107.65)
+		(width 0.5)
+		(layer "B.Cu")
 		(net "PSI")
 	)
 	(segment
-		(start 127.312233 110.15)
-		(end 129.15 110.15)
-		(width 0.5)
-		(layer "F.Cu")
+		(start 144.773688 112.73)
+		(end 146.127767 112.73)
+		(width 0.5)
+		(layer "B.Cu")
 		(net "PSI")
 	)
 	(segment
-		(start 126.575 109.412767)
-		(end 126.575 89.835)
-		(width 0.5)
-		(layer "F.Cu")
-		(net "PSI")
-	)
-	(segment
-		(start 152.212 110.022)
-		(end 152.212 111.852027)
-		(width 0.5)
-		(layer "F.Cu")
-		(net "PSI")
-	)
-	(segment
-		(start 152.212 111.852027)
-		(end 151.502027 112.562)
-		(width 0.5)
-		(layer "F.Cu")
-		(net "PSI")
-	)
-	(segment
-		(start 148.539767 112.562)
-		(end 148.406767 112.695)
-		(width 0.5)
-		(layer "F.Cu")
-		(net "PSI")
-	)
-	(segment
-		(start 151.502027 112.562)
-		(end 148.539767 112.562)
-		(width 0.5)
-		(layer "F.Cu")
-		(net "PSI")
-	)
-	(segment
-		(start 126.575 89.835)
-		(end 127.83 88.58)
-		(width 0.5)
-		(layer "F.Cu")
+		(start 149.84 107.65)
+		(end 145.092233 107.65)
+		(width 0.5)
+		(layer "B.Cu")
 		(net "PSI")
 	)
@@
 	)
 	(segment
+		(start 128.51 104.5)
+		(end 127.83 103.82)
+		(width 0.5)
+		(layer "B.Cu")
+		(net "PSO")
+	)
+	(segment
 		(start 130 104.5)
-		(end 130 85.67)
+		(end 128.51 104.5)
 		(width 0.5)
 		(layer "B.Cu")
@@
 	)
 	(segment
-		(start 130 85.67)
-		(end 127.83 83.5)
+		(start 130 104.5)
+		(end 130 90.75)
 		(width 0.5)
 		(layer "B.Cu")
 		(net "PSO")
+	)
+	(segment
+		(start 127.83 88.58)
+		(end 130 90.75)
+		(width 0.5)
+		(layer "B.Cu")
+		(net "PSO")
+	)
+	(segment
+		(start 151.854109 113.412)
+		(end 153.5 111.766109)
+		(width 0.8)
+		(layer "F.Cu")
+		(net "OPT_1")
+	)
+	(segment
+		(start 145.61 126.68)
+		(end 151.854109 120.435891)
+		(width 0.8)
+		(layer "F.Cu")
+		(net "OPT_1")
 	)
 	(segment
@@
 	)
 	(segment
-		(start 153.5 112)
-		(end 148.98 116.52)
+		(start 151.854109 120.435891)
+		(end 151.854109 113.412)
 		(width 0.8)
 		(layer "F.Cu")
@@
 	(segment
 		(start 153.5 90.999999)
-		(end 153.5 112)
-		(width 0.8)
-		(layer "F.Cu")
-		(net "OPT_1")
-	)
-	(segment
-		(start 148.98 116.52)
-		(end 145.61 116.52)
-		(width 0.8)
-		(layer "F.Cu")
+		(end 153.5 111.766109)
+		(width 0.8)
+		(layer "F.Cu")
