File: mb_adv_1.0.kicad_sch (KiCad schematic)
At the start: 5 parts, among them SW2 SW_SP3T, U2 gba_link_cable, U3 BOB-12009

Commit message: update README.md, schematic, and pcb
Connections:
- net PSI: now also A1.4 (GPIO2); no longer A1.2 (GPIO1)
- net PSO: now also A1.2 (GPIO1); no longer A1.4 (GPIO2)
Changed lines of the file:
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@@
-	(wire
-		(pts
-			(xy 50.8 80.01) (xy 54.61 80.01)
-		)
-		(stroke
-			(width 0)
-			(type default)
-		)
-	)
 	(wire
 		(pts
@@
 	(wire
 		(pts
+			(xy 49.53 80.01) (xy 54.61 80.01)
+		)
+		(stroke
+			(width 0)
+			(type default)
+		)
+	)
+	(wire
+		(pts
 			(xy 50.8 77.47) (xy 54.61 77.47)
 		)
@@
 		)
 	)
-	(global_label "PSO"
-		(shape input)
-		(at 50.8 80.01 180)
+	(global_label "HV"
+		(shape output)
+		(at 170.18 44.45 0)
+		(fields_autoplaced yes)
+		(effects
+			(font
+				(size 1.27 1.27)
+			)
+			(justify left)
+		)
+		(property "Intersheetrefs" "${INTERSHEET_REFS}"
+			(at 175.5843 44.45 0)
+			(hide yes)
+			(show_name no)
+			(do_not_autoplace no)
+			(effects
+				(font
+					(size 1.27 1.27)
+				)
+				(justify left)
+			)
+		)
+	)
+	(global_label "LV"
+		(shape output)
+		(at 242.57 59.69 0)
+		(fields_autoplaced yes)
+		(effects
+			(font
+				(size 1.27 1.27)
+			)
+			(justify left)
+		)
+		(property "Intersheetrefs" "${INTERSHEET_REFS}"
+			(at 247.6719 59.69 0)
+			(hide yes)
+			(show_name no)
+			(do_not_autoplace no)
+			(effects
+				(font
+					(size 1.27 1.27)
+				)
+				(justify left)
+			)
+		)
+	)
+	(global_label "OPT_2"
+		(shape output)
+		(at 217.17 111.76 0)
+		(fields_autoplaced yes)
+		(effects
+			(font
+				(size 1.27 1.27)
+			)
+			(justify left)
+		)
+		(property "Intersheetrefs" "${INTERSHEET_REFS}"
+			(at 226.3238 111.76 0)
+			(hide yes)
+			(show_name no)
+			(do_not_autoplace no)
+			(effects
+				(font
+					(size 1.27 1.27)
+				)
+				(justify left)
+			)
+		)
+	)
+	(global_label "HV"
+		(shape output)
+		(at 199.39 59.69 180)
 		(fields_autoplaced yes)
 		(effects
@@
 		)
 		(property "Intersheetrefs" "${INTERSHEET_REFS}"
-			(at 44.0048 80.01 0)
+			(at 193.9857 59.69 0)
 			(hide yes)
 			(show_name no)
@@
 		)
 	)
-	(global_label "HV"
-		(shape output)
-		(at 170.18 44.45 0)
-		(fields_autoplaced yes)
-		(effects
-			(font
-				(size 1.27 1.27)
-			)
-			(justify left)
-		)
-		(property "Intersheetrefs" "${INTERSHEET_REFS}"
-			(at 175.5843 44.45 0)
-			(hide yes)
-			(show_name no)
-			(do_not_autoplace no)
-			(effects
-				(font
-					(size 1.27 1.27)
-				)
-				(justify left)
-			)
-		)
-	)
-	(global_label "LV"
-		(shape output)
-		(at 242.57 59.69 0)
-		(fields_autoplaced yes)
-		(effects
-			(font
-				(size 1.27 1.27)
-			)
-			(justify left)
-		)
-		(property "Intersheetrefs" "${INTERSHEET_REFS}"
-			(at 247.6719 59.69 0)
-			(hide yes)
-			(show_name no)
-			(do_not_autoplace no)
-			(effects
-				(font
-					(size 1.27 1.27)
-				)
-				(justify left)
-			)
-		)
-	)
-	(global_label "OPT_2"
-		(shape output)
-		(at 217.17 111.76 0)
-		(fields_autoplaced yes)
-		(effects
-			(font
-				(size 1.27 1.27)
-			)
-			(justify left)
-		)
-		(property "Intersheetrefs" "${INTERSHEET_REFS}"
-			(at 226.3238 111.76 0)
-			(hide yes)
-			(show_name no)
-			(do_not_autoplace no)
-			(effects
-				(font
-					(size 1.27 1.27)
-				)
-				(justify left)
-			)
-		)
-	)
-	(global_label "HV"
-		(shape output)
-		(at 199.39 59.69 180)
+	(global_label "PSI"
+		(shape output)
+		(at 49.53 80.01 180)
 		(fields_autoplaced yes)
 		(effects
@@
 		)
 		(property "Intersheetrefs" "${INTERSHEET_REFS}"
-			(at 193.9857 59.69 0)
-			(hide yes)
-			(show_name no)
-			(do_not_autoplace no)
-			(effects
-				(font
-					(size 1.27 1.27)
-				)
-				(justify right)
-			)
-		)
-	)
-	(global_label "PSI"
-		(shape output)
-		(at 50.8 77.47 180)
-		(fields_autoplaced yes)
-		(effects
-			(font
-				(size 1.27 1.27)
-			)
-			(justify right)
-		)
-		(property "Intersheetrefs" "${INTERSHEET_REFS}"
-			(at 44.7305 77.47 0)
+			(at 43.4605 80.01 0)
 			(hide yes)
 			(show_name no)
@@
 			)
 		)
+	)
+	(global_label "PSO"
+		(shape input)
+		(at 50.8 77.47 180)
+		(fields_autoplaced yes)
+		(effects
+			(font
+				(size 1.27 1.27)
+			)
+			(justify right)
+		)
+		(property "Intersheetrefs" "${INTERSHEET_REFS}"
+			(at 44.0048 77.47 0)
+			(hide yes)
+			(show_name no)
+			(do_not_autoplace no)
+			(effects
+				(font
+					(size 1.27 1.27)
+				)
+				(justify right)
+			)
+		)

Commit message: update pinout
Connections:
- net OPT_1: now also A1.22 (GPIO17); no longer A1.26 (GPIO20)
- net PSC: now also A1.9 (GPIO6)
- net PSD: now also A1.7 (GPIO5)
- net PSI: now also A1.2 (GPIO1), A1.26 (GPIO20); no longer A1.4 (GPIO2)
- net PSO: now also A1.10 (GPIO7), A1.4 (GPIO2); no longer A1.2 (GPIO1)
Changed lines of the file:
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@@
 	(title_block
 		(title "mb_adv")
-		(date "2026-09-27")
+		(date "2026-09-28")
 		(rev "1.0")
 		(company "aestellic")
@@
 	(wire
 		(pts
+			(xy 100.33 80.01) (xy 104.14 80.01)
+		)
+		(stroke
+			(width 0)
+			(type default)
+		)
+	)
+	(wire
+		(pts
 			(xy 170.18 57.15) (xy 170.18 66.04)
 		)
@@
 	(wire
 		(pts
+			(xy 49.53 90.17) (xy 54.61 90.17)
+		)
+		(stroke
+			(width 0)
+			(type default)
+		)
+	)
+	(wire
+		(pts
 			(xy 50.8 82.55) (xy 54.61 82.55)
 		)
@@
 	(wire
 		(pts
+			(xy 50.8 80.01) (xy 54.61 80.01)
+		)
+		(stroke
+			(width 0)
+			(type default)
+		)
+	)
+	(wire
+		(pts
 			(xy 63.5 40.64) (xy 64.77 40.64)
 		)
@@
 	(wire
 		(pts
+			(xy 49.53 92.71) (xy 54.61 92.71)
+		)
+		(stroke
+			(width 0)
+			(type default)
+		)
+	)
+	(wire
+		(pts
 			(xy 191.77 111.76) (xy 199.39 111.76)
 		)
@@
 	(wire
 		(pts
+			(xy 105.41 87.63) (xy 100.33 87.63)
+		)
+		(stroke
+			(width 0)
+			(type default)
+		)
+	)
+	(wire
+		(pts
 			(xy 100.33 92.71) (xy 104.14 92.71)
 		)
@@
 	(wire
 		(pts
-			(xy 100.33 87.63) (xy 104.14 87.63)
-		)
-		(stroke
-			(width 0)
-			(type default)
-		)
-	)
-	(wire
-		(pts
 			(xy 72.39 40.64) (xy 72.39 52.07)
 		)
@@
 	(wire
 		(pts
+			(xy 50.8 87.63) (xy 54.61 87.63)
+		)
+		(stroke
+			(width 0)
+			(type default)
+		)
+	)
+	(wire
+		(pts
 			(xy 237.49 46.99) (xy 242.57 46.99)
 		)
@@
 	(wire
 		(pts
-			(xy 49.53 80.01) (xy 54.61 80.01)
-		)
-		(stroke
-			(width 0)
-			(type default)
-		)
-	)
-	(wire
-		(pts
-			(xy 50.8 77.47) (xy 54.61 77.47)
+			(xy 49.53 77.47) (xy 54.61 77.47)
 		)
 		(stroke
@@
 		)
 	)
+	(global_label "PSI"
+		(shape output)
+		(at 105.41 87.63 0)
+		(fields_autoplaced yes)
+		(effects
+			(font
+				(size 1.27 1.27)
+			)
+			(justify left)
+		)
+		(property "Intersheetrefs" "${INTERSHEET_REFS}"
+			(at 111.4795 87.63 0)
+			(hide yes)
+			(show_name no)
+			(do_not_autoplace no)
+			(effects
+				(font
+					(size 1.27 1.27)
+				)
+				(justify left)
+			)
+		)
+	)
 	(global_label "OPT_2"
 		(shape output)
@@
 	(global_label "PSI"
 		(shape output)
-		(at 49.53 80.01 180)
+		(at 49.53 77.47 180)
 		(fields_autoplaced yes)
 		(effects
@@
 		)
 		(property "Intersheetrefs" "${INTERSHEET_REFS}"
-			(at 43.4605 80.01 0)
+			(at 43.4605 77.47 0)
 			(hide yes)
 			(show_name no)
@@
 		)
 	)
+	(global_label "PSO"
+		(shape input)
+		(at 50.8 80.01 180)
+		(fields_autoplaced yes)
+		(effects
+			(font
+				(size 1.27 1.27)
+			)
+			(justify right)
+		)
+		(property "Intersheetrefs" "${INTERSHEET_REFS}"
+			(at 44.0048 80.01 0)
+			(hide yes)
+			(show_name no)
+			(do_not_autoplace no)
+			(effects
+				(font
+					(size 1.27 1.27)
+				)
+				(justify right)
+			)
+		)
+	)
 	(global_label "OPT_3"
 		(shape input)
@@
 		)
 	)
-	(global_label "OPT_1"
-		(shape input)
-		(at 104.14 87.63 0)
-		(fields_autoplaced yes)
-		(effects
-			(font
-				(size 1.27 1.27)
-			)
-			(justify left)
-		)
-		(property "Intersheetrefs" "${INTERSHEET_REFS}"
-			(at 112.8704 87.63 0)
-			(hide yes)
-			(show_name no)
-			(do_not_autoplace no)
-			(effects
-				(font
-					(size 1.27 1.27)
-				)
-				(justify left)
-			)
-		)
-	)
 	(global_label "OPT_2"
 		(shape input)
@@
 		)
 	)
+	(global_label "OPT_1"
+		(shape input)
+		(at 104.14 80.01 0)
+		(fields_autoplaced yes)
+		(effects
+			(font
+				(size 1.27 1.27)
+			)
+			(justify left)
+		)
+		(property "Intersheetrefs" "${INTERSHEET_REFS}"
+			(at 112.8704 80.01 0)
+			(hide yes)
+			(show_name no)
+			(do_not_autoplace no)
+			(effects
+				(font
+					(size 1.27 1.27)
+				)
+				(justify left)
+			)
+		)
+	)
 	(global_label "PSD"
 		(shape bidirectional)
@@
 		)
 	)
+	(global_label "PSD"
+		(shape bidirectional)
+		(at 50.8 87.63 180)
+		(fields_autoplaced yes)
+		(effects
+			(font
+				(size 1.27 1.27)
+			)
+			(justify right)
+		)
+		(property "Intersheetrefs" "${INTERSHEET_REFS}"
+			(at 42.954 87.63 0)
+			(hide yes)
+			(show_name no)
+			(do_not_autoplace no)
+			(effects
+				(font
+					(size 1.27 1.27)
+				)
+				(justify right)
+			)
+		)
+	)
+	(global_label "PSC"
+		(shape input)
+		(at 49.53 90.17 180)
+		(fields_autoplaced yes)
+		(effects
+			(font
+				(size 1.27 1.27)
+			)
+			(justify right)
+		)
+		(property "Intersheetrefs" "${INTERSHEET_REFS}"
+			(at 42.7953 90.17 0)
+			(hide yes)
+			(show_name no)
+			(do_not_autoplace no)
+			(effects
+				(font
+					(size 1.27 1.27)
+				)
+				(justify right)
+			)
+		)
+	)
 	(global_label "PSC"
 		(shape output)
@@
 	(global_label "PSO"
 		(shape input)
-		(at 50.8 77.47 180)
+		(at 49.53 92.71 180)
 		(fields_autoplaced yes)
 		(effects
@@
 		)
 		(property "Intersheetrefs" "${INTERSHEET_REFS}"
-			(at 44.0048 77.47 0)
-			(hide yes)
-			(show_name no)
+			(at 42.7348 92.71 0)
+			(hide yes)
+			(show_name no)

Commit message: add microSD card
Parts:
- added U1: Adafruit-MicroSD-SPI-4682, adafruit:adafruit_4682, symbol adafruit_4682:microSD_SPI_SDIO_4682
Connections:
- net GND: now also U1.2 (GND)
- net HV: now also D1.2 (A)
- net LV: now also A1.36 (3V3), U1.1 (3V); no longer D1.2 (A)
- net PSC: no longer A1.9 (GPIO6)
- net PSD: no longer A1.7 (GPIO5)
- net PSI: no longer A1.26 (GPIO20)
- net PSO: no longer A1.10 (GPIO7)
- new net uSC: A1.9 (GPIO6), U1.3 (CLK)
- new net uSD: A1.7 (GPIO5), U1.6 (CS)
- new net uSI: A1.26 (GPIO20), U1.5 (SI)
- new net uSO: A1.10 (GPIO7), U1.4 (SO)
Other:
- note added: "microSD SPI"
- moved on the sheet: D1, SW2
